Commit message: camera and laser plugin added

File: install/ack_robot_description/share/ack_robot_description/urdf/traktor.urdf (robot description, URDF)
Before this commit: robot traktor, 10 links, 9 joints
Links:
- added link camera_link, mass 0.1; collision box size=0.025 0.1 0.025; visual box size=0.025 0.1 0.025
Joints:
- added joint base_to_camera: type fixed, parent base_link, child camera_link, origin xyz=0 -0.3 1.2 rpy=0 0 1.5707

Commit message: laser fixed

File: install/ack_robot_description/share/ack_robot_description/urdf/traktor.urdf (robot description, URDF)
Before this commit: robot ackerman_robot, 11 links, 10 joints
Links:
- removed link camera_link
- link laser_link: geometry collision cylinder length=0.04 radius=0.05; visual cylinder length=0.04 radius=0.05
Joints:
- removed joint base_to_camera
- joint gps_joint: origin xyz=0.0 0.0 0.5 rpy=0.0 0.0 0.0 -> xyz=0.0 0.0 0 rpy=0.0 0.0 0.0
- joint imu_joint: origin xyz=1.0 0.0 0.5 rpy=0.0 0.0 0.0 -> xyz=1.0 0.0 0 rpy=0.0 0.0 0.0
- joint laser_joint: axis 0.0 0.0 0.0 -> (none); child laser_link -> laser_frame; limit lower=0.0 upper=0.0 effort=0.0 velocity=0.0 -> (none); origin xyz=0.0 0.0 0.0 rpy=0.0 0.0 0.0 -> xyz=1 0 0.51 rpy=0.0 0.0 0.0; type revolute -> fixed

Commit message: display.xml update

File: install/ack_robot_description/share/ack_robot_description/urdf/traktor.urdf (robot description, URDF)
Before this commit: robot ackerman_robot, 10 links, 9 joints
Links:
- removed link laser_link
- added link hokuyo_link, mass 1e-5; collision cylinder length=0.05 radius=0.05; visual cylinder length=0.05 radius=0.05
Joints:
- removed joint laser_joint
- added joint hokuyo_joint: type fixed, parent base_link, child hokuyo_link, origin xyz=1 0 0.51 rpy=0 0 0, axis 0 1 0
