Commit message: tf_frame added

File: src/ack_robot_description/urdf/traktor.urdf (robot description, URDF)
Before this commit: robot ackerman_robot, 10 links, 9 joints
Links:
- link sag_arka: geometry collision cylinder length=0.20 radius=0.4; visual cylinder length=0.20 radius=0.4
- link sag_on_teker: geometry collision cylinder length=0.20 radius=0.25; visual cylinder length=0.20 radius=0.25
- link sol_arka: geometry collision cylinder length=0.20 radius=0.4; visual cylinder length=0.20 radius=0.4
- link sol_on_teker: geometry collision cylinder length=0.20 radius=0.25; visual cylinder length=0.20 radius=0.25
